File: Hardware/pcb_file.brd (EAGLE design)
At the start: 170.2 x 111.2 mm, 103 parts, among them IC1 BD5229G-TR, IC4 XC6220A331MR-G, J1 FH34SRJ-24S-0.5SH_99_, J2 SAMACSYS_PARTS_USB4110-GF-A, J3 QWIIC_RIGHT_ANGLE, J4 112A-TAAR-R03_ATTEND, Q1 20V/4.2A/52mΩ/1.4W, Q2 20V/4.2A/52mΩ/1.4W, Q3 SI1308EDL-T1-GE3, U1 W25Q512JVEIQ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

Commit message: Fixed issues
Parts:
- renumbered TP5 to TPGND
Routing:
- net GND: track 822.8 -> 894.2 mm, vias 14 -> 18
- net MISO: track 98.0 -> 130.8 mm
- net SDA: track 204.3 -> 235.4 mm
- net EPD_DC: track 131.8 -> 112.5 mm, vias 4 -> 5
- net IO/CHANGE: track 60.6 -> 76.6 mm
- net SCK: track 197.4 -> 213.1 mm, vias 6 -> 7
- net N$13: track 31.2 -> 15.5 mm
- net 3V3: track 485.3 -> 470.0 mm
- net I2C_PW: track 166.8 -> 181.1 mm
- net EPD_RST: track 103.0 -> 117.0 mm
- net 32KHZ: track 93.8 -> 106.0 mm
- net SS_SD: track 98.7 -> 110.7 mm, vias 5 -> 2
- net VBUS: track 137.2 -> 129.6 mm
- net MOSI: track 202.4 -> 209.9 mm
- net SCL: track 218.0 -> 225.2 mm, vias 6 -> 7
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